File: rfid.kicad_sch (KiCad schematic)
At the start: 0 parts

Commit message: Add RFID circuit.
Parts:
- added C19, C20, C21, C22, C23, C24: C, symbol Device:C
- added L2, L3: L, symbol Device:L
- added NT1, NT2, NT3, NT4, NT5: NetTie_2, symbol Device:NetTie_2
- added U2: PN5120A0HN1, Package_DFN_QFN:HVQFN-32-1EP_5x5mm_P0.5mm_EP3.1x3.1mm, symbol RF_RFID:PN5120A0HN1
Connections:
- new net: C22.2, C24.2, NT5.1
- new net: NT4.1, NT5.2
- new net: NT3.1, NT4.2
- new net: L2.1, L3.1
- new net: C20.2, C22.1, L3.2
- new net: C19.1, C21.1, L2.2
- new net GND: C19.2, C20.1, C23.2, C24.1, U2.10 (TVSS), U2.14 (TVSS)
- new net TURN1A: C21.2, C23.1, NT1.2
- new net TURN1B: NT1.1, NT2.2
- new net TURN2A: NT2.1, NT3.2
