File: DS18B20_Breakout_Board.kicad_sch (KiCad schematic)
At the start: 4 parts, among them J2 Conn_01x03_Socket, J3 Conn_01x03_Socket, U2 DS18B20

Commit message: Update sheet naming
Other:
- company: (none) -> Alister, Damien, Nils
- title: (none) -> CC3501 Design Project
Changed lines of the file:
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@@
 	(generator_version "10.0")
 	(paper "A4")
+	(title_block
+		(title "CC3501 Design Project")
+		(date "2026-06-22")
+		(rev "1")
+		(company "Alister, Damien, Nils")
+	)
 	(text_box "DS18B20 configured in parasitic power mode. FET and pull-up resistor to be placed on the mainboard close to the GPIO pin."
 		(exclude_from_sim no)
