File: load_cell.kicad_sch (KiCad schematic)
At the start: 17 parts, among them J7 Conn_01x04, Q1 SS8550, U7 HX711

Commit message: Update sheet naming
Other:
- company: (none) -> Alister, Damien, Nils
- title: (none) -> CC3501 Design Project
Changed lines of the file:
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@@
 	(generator_version "10.0")
 	(paper "A4")
+	(title_block
+		(title "CC3501 Design Project")
+		(date "2026-06-22")
+		(rev "1")
+		(company "Alister, Damien, Nils")
+	)
 	(text "E+\nE-\nS-\nS+\n"
 		(exclude_from_sim no)

Commit message: ALL the PCB edits.
Parts:
- added JP5: SolderJumper_2_Bridged, Jumper:SolderJumper-2_P1.3mm_Bridged2Bar_RoundedPad1.0x1.5mm, symbol Jumper:SolderJumper_2_Bridged
- L4: value 3.3uH -> L; footprint Inductor_SMD:L_0805_2012Metric -> Inductor_THT:L_Axial_L11.0mm_D4.5mm_P15.24mm_Horizontal_Fastron_MECC; LCSC PN C53063751 -> (none); now not fitted; now left out of the parts list
Connections:
- net at C21.2, C39.1, J7.1 (Pin_1)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: now also JP5.2 (B)
- net at L4.2, Q1.3 (C), R16.1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: now also JP5.1 (A)
