File: tft_display.kicad_sch (KiCad schematic)
At the start: 9 parts, among them J5 Conn_01x04_Socket, J6 Conn_01x08_Socket, J8 Conn_01x06_Socket, Q3 AO3401A

Commit message: ALL the PCB edits.
Parts:
- R13: LCSC PN C25190 -> C4177
Changed lines of the file:
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@@
 			)
 		)
-		(property "LCSC PN" "C25190"
+		(property "LCSC PN" "C4177"
 			(at 211.582 74.422 0)
 			(show_name no)

Commit message: changed component footprint
Parts:
- R13: footprint Resistor_SMD:R_0201_0603Metric -> Resistor_SMD:R_0603_1608Metric
Changed lines of the file:
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@@
 			)
 		)
-		(property "Footprint" "Resistor_SMD:R_0201_0603Metric"
+		(property "Footprint" "Resistor_SMD:R_0603_1608Metric"
 			(at 220.472 74.93 90)
 			(hide yes)
