File: RFID/CE-PiicoDev-RFID-Reader-Writer.kicad_sch (KiCad schematic)
At the start: 32 parts, among them U3 MFRC522, Y2 Crystal_GND23

Commit message: Add symbol/footprint library linkages.
Parts:
- Y2: LCSC PN (none) -> C113669
Changed lines of the file:
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@@
 			)
 		)
-		(property "LCSC PN" ""
+		(property "LCSC PN" "C113669 "
 			(at 187.96 104.14 0)
 			(hide yes)

Commit message: Update sheet naming
Other:
- company: Core Electronics -> Alister, Damien, Nils
- title: PiicoDev RFID Module -> CC3501 Design Project
Changed lines of the file:
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@@
 	(paper "A4")
 	(title_block
-		(title "PiicoDev RFID Module")
-		(date "2022-01-12")
-		(rev "10")
-		(company "Core Electronics")
+		(title "CC3501 Design Project")
+		(date "2026-06-22")
+		(rev "1")
+		(company "Alister, Damien, Nils")
 		(comment 1 "Designed at Core Electronics by Peter Johnston")
 		(comment 2 "PiicoDev and the PiicoDev logo are trademarks of Core Electronics Pty Ltd.")
