File: RFID/CE-PiicoDev-RFID-Reader-Writer.kicad_sch (KiCad schematic)
At the start: 32 parts, among them U3 MFRC522, Y2 Crystal_GND23

Commit message: ALL the PCB edits.
Parts:
- added C43, C44: 30pF, Capacitor_SMD:C_0201_0603Metric, symbol Device:C
- added C45, C46: 10p, Capacitor_SMD:C_0402_1005Metric, symbol Device:C
- added C47, C49: 220pF, Capacitor_SMD:C_0402_1005Metric, symbol Device:C
- added C48, C50: 47pF, Capacitor_SMD:C_0402_1005Metric, symbol Device:C
- C23, C24: value 22p NP0 -> 22pF C0G ±5%; LCSC PN C106203 -> C1555
- C25, C26: value 62p NP0 2% -> 33pF; footprint Capacitor_SMD:C_0805_2012Metric -> Capacitor_SMD:C_0402_1005Metric; LCSC PN C520069 -> C1562
- C27, C28: value 56p -> 47p; footprint Capacitor_SMD:C_0603_1608Metric -> Capacitor_SMD:C_0402_1005Metric; LCSC PN C107053 -> C1567
- C29, C30: value 270p NP0 2% -> 220pF; footprint Capacitor_SMD:C_0603_1608Metric -> Capacitor_SMD:C_0402_1005Metric; LCSC PN C327196 -> C1530
- C31, C32: value 270p NP0 2% -> 47pF; footprint Capacitor_SMD:C_0603_1608Metric -> Capacitor_SMD:C_0402_1005Metric; LCSC PN C327196 -> C1567
- C34: value 1n NP0 10% -> 1nF X7R ±10%; LCSC PN C106246 -> C1588
- L2, L3: footprint Inductor_SMD:L_0603_1608Metric -> Inductor_SMD:L_0805_2012Metric
- U3: value MFRC522 -> MFRC52202HN(TOKMAS)
Connections:
- net GND: now also C26.1, C43.2, C44.1, C47.2, C48.2, C49.1, C50.1; no longer C26.2
- net TURN1A: now also C45.1, C49.2, C50.2
- net TURN6B: now also C46.1, C47.1, C48.1
- net at C25.1, C27.2, L3.2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: now also C43.1, C46.2
- net at C28.2, L2.2: now also C26.2, C44.2, C45.2; no longer C26.1
Other:
- moved on the sheet: C25, C31, C32

Commit message: changed component footprint
Parts:
- C43, C44: footprint Capacitor_SMD:C_0201_0603Metric -> Capacitor_SMD:C_0603_1608Metric
Changed lines of the file:
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@@
 			)
 		)
-		(property "Footprint" "Capacitor_SMD:C_0201_0603Metric"
+		(property "Footprint" "Capacitor_SMD:C_0603_1608Metric"
 			(at 211.7852 87.63 0)
 			(hide yes)
@@
 			)
 		)
-		(property "Footprint" "Capacitor_SMD:C_0201_0603Metric"
+		(property "Footprint" "Capacitor_SMD:C_0603_1608Metric"
 			(at 211.7852 78.74 0)
 			(hide yes)
